File: pcb/mouse-pcb.kicad_sch (KiCad schematic)
At the start: 45 parts, among them J1 TYPE-C-31-M-12, SW1 D2FC-F-7N20M, SW2 D2FC-F-7N20M, SW3 D2FC-F-7N20M, U1 PAW3395-T6QU, U2 NRF52840-QIAA-R7, Y1 32MHz, Y2 32.768kHz

Commit message: feat: impedance calcualated
JLC04161H-3313(finished thicknes1.56mm+-10%
50 ohm 6.16 mil width (antenna)
90 ohm 4.4 mil width 4.0 mil spacing (differential pair)
Connections:
- net SCLK: now also U2.L24 (P0.09/NFC1)
Other:
- moved on the sheet: SW1
Changed lines of the file:
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@@
 	(global_label "SCLK"
 		(shape input)
-		(at 140.97 165.1 180)
+		(at 143.51 168.91 180)
 		(fields_autoplaced yes)
 		(effects
@@
 		)
 		(property "Intersheetrefs" "${INTERSHEET_REFS}"
-			(at 133.2072 165.1 0)
+			(at 135.7472 168.91 0)
 			(hide yes)
 			(show_name no)
@@
 	(symbol
 		(lib_id "mouse_library:D2FC-F-7N20M")
-		(at 455.93 184.15 0)
+		(at 280.67 190.5 0)
 		(unit 1)
 		(body_style 1)
@@
 		(fields_autoplaced yes)
 		(property "Reference" "SW1"
-			(at 477.52 172.72 0)
+			(at 302.26 179.07 0)
 			(show_name no)
 			(do_not_autoplace no)
@@
 		)
 		(property "Value" "D2FC-F-7N20M"
-			(at 477.52 175.26 0)
+			(at 302.26 181.61 0)
 			(show_name no)
 			(do_not_autoplace no)
@@
 		)
 		(property "Footprint" "mouse_library:SW_D2FC_OMR"
-			(at 457.2 179.07 0)
+			(at 281.94 185.42 0)
 			(hide yes)
 			(show_name no)
@@
 		)
 		(property "Datasheet" "https://www.lcsc.com/datasheet/C5157566.pdf"
-			(at 457.2 179.07 0)
+			(at 281.94 185.42 0)
 			(hide yes)
 			(show_name no)
@@
 		)
 		(property "Description" ""
-			(at 455.93 184.15 0)
+			(at 280.67 190.5 0)
 			(hide yes)
 			(show_name no)
@@
 		)
 		(property "MPN" "D2FC-F-7N(20M)"
-			(at 455.93 184.15 0)
+			(at 280.67 190.5 0)
 			(hide yes)
 			(show_name no)
@@
 		)
 		(property "LCSC_PART_NUMBER" "C5157566"
-			(at 455.93 184.15 0)
+			(at 280.67 190.5 0)
 			(hide yes)
 			(show_name no)

Commit message: feat: usblc6 added
Parts:
- added U3: USBLC6-2SC6, Package_TO_SOT_SMD:SOT-23-6, symbol Power_Protection:USBLC6-2SC6
- SW1: value D2FC-F-7N20M -> left click
- SW2: value D2FC-F-7N20M -> center click
- SW3: value D2FC-F-7N20M -> right click
Connections:
- net +3V3: now also SW1.1 (COM), SW2.1 (COM), SW3.1 (COM)
- net LCLIKC: now reaches SW1.2 (NO)
- net LCLIKC: now also U2.AD22 (P1.00)
- net RCLICK: now reaches SW3.2 (NO)
- net RCLICK: now also U2.AD18 (P0.22)
- net CCLICK: now reaches SW2.2 (NO)
- net CCLICK: now also U2.AD20 (P0.24)
- no-connect marks 41 -> 40
Other:
- note added: "Clicks"
- moved on the sheet: J1, SW1, SW2, SW3

Commit message: feat: battery management added, mcu circuits are ready
Parts:
- added C28: 1.0uF, Capacitor_SMD:C_0402_1005Metric, symbol Device:C
- added C29: 10uF, Capacitor_SMD:C_0402_1005Metric, symbol Device:C
- added J2: Conn_01x02, Connector_JST:JST_SHL_SM02B-SHLS-TF_1x02-1MP_P1.00mm_Horizontal, symbol Connector_Generic:Conn_01x02
- added R3, R4: 5.1K, Capacitor_SMD:C_0805_2012Metric, symbol Device:R_US
- added R5: 10K, Capacitor_SMD:C_0402_1005Metric, symbol Device:R_US
- added R6, R7: 4.7K, Capacitor_SMD:C_0402_1005Metric, symbol Device:R_US
- added U4: BQ25180YBGR, mouse_library:IC_BQ25180YBGR, symbol mouse_library:BQ25180YBGR
- C24, C25: footprint Capacitor_SMD:C_0402_1005Metric -> Capacitor_SMD:C_0201_0603Metric
- R1: footprint Resistor_SMD:R_0805_2012Metric -> Capacitor_SMD:C_0805_2012Metric
Connections:
- net +3V3: now also R6.1, R7.1
- net D+: now also U3.4 (I/O2)
- net D-: now also U3.6 (I/O1)
- net GND: now also J1.S1 (SHIELD), J1.S2 (SHIELD), J1.S3 (SHIELD), J1.S4 (SHIELD), U3.2 (GND), C28.1, C29.2, J2.1 (Pin_1), R3.2, R4.1, R5.2, U4.D2 (GND)
- net MISO: now also U2.L1 (P0.06); no longer U2.U24 (P1.04)
- net MOSI: now also U2.N1 (P0.08); no longer U2.R24 (P1.06)
- net MOTION: now also U2.U1 (P0.12); no longer U2.J24 (P0.10/NFC2)
- net NCS: now also U2.J1 (P0.04/AIN2); no longer U2.R1 (P1.09)
- net NRESET: now also U2.G1 (P0.26); no longer U2.W24 (P1.02)
- net SCLK: now also U2.R1 (P1.09); no longer U2.L24 (P0.09/NFC1)
- net VBUS: now also U3.5 (VBUS), C28.2, U4.A2 (IN)
- net VDDH: now also C29.1, U4.B2 (SYS)
- net at J1.A5 (CC1): now also R4.2
- net USB D+: now reaches J1.A6 (DP1)
- net USB D+: now also J1.B6 (DP2), U3.3 (I/O2)
- net USB D-: now reaches J1.A7 (DN1)
- net USB D-: now also J1.B7 (DN2), U3.1 (I/O1)
- net at J1.B5 (CC2): now also R3.1
- net SCL: now reaches U2.A10 (P0.29/AIN5)
- net SCL: now also R6.2, U4.B1 (SCL)
- net SDA: now reaches U2.A12 (P0.02/AIN0)
- net SDA: now also R7.2, U4.C1 (SDA)
- new net: R5.1, U4.D1 (TS/MR)
- new net INT_BAT: U4.A1 (~{INT})
- new net VBAT: J2.2 (Pin_2), U4.C2 (BAT)
- no-connect marks 40 -> 35
Other:
- note added: "BATTERY MNGMNT"
- note added: "USB"
- note added: "pairing button"
- note added: "resistor for i2c"
- note added: "status rgb"
- note added: "switch 2.4 ble"
- note removed: "Battery Management IC — TI BQ25180"
- note removed: "USBLC6-2SC6"
- note removed: "circuits mcu"
- moved on the sheet: C23, C24, C25, J1, L6, U3, VR1
